Commit message: Separate Robotiq geometry from URCap and USB hardware control

File: urdf/robotiq_gripper.ros2_control.xacro (robot description, xacro)
@@ -1,19 +1,31 @@
 <?xml version="1.0"?>
 <robot xmlns:xacro="http://www.ros.org/wiki/xacro">
-    <xacro:macro name="robotiq_gripper_ros2_control" params="name com_port">
+    <xacro:macro name="robotiq_gripper_ros2_control" params="name com_port tf_prefix:='' use_fake_hardware:=false">
         <ros2_control name="${name}" type="system">
             <hardware>
-                <plugin>robotiq_driver/RobotiqGripperHardwareInterface</plugin>
-                <param name="gripper_closed_position">0.7929</param>
-                <param name="COM_port">${com_port}</param>
-                <param name="gripper_speed_multiplier">1.0</param>
-                <param name="gripper_force_multiplier">0.5</param>
+                <xacro:if value="${use_fake_hardware}">
+                    <plugin>mock_components/GenericSystem</plugin>
+                </xacro:if>
+                <xacro:unless value="${use_fake_hardware}">
+                    <plugin>robotiq_driver/RobotiqGripperHardwareInterface</plugin>
+                    <param name="gripper_closed_position">0.7929</param>
+                    <param name="COM_port">${com_port}</param>
+                    <param name="gripper_speed_multiplier">1.0</param>
+                    <param name="gripper_force_multiplier">0.5</param>
+                </xacro:unless>
             </hardware>
-            <joint name="robotiq_85_left_knuckle_joint">
-                <param name="initial_position">0.7929</param>
+            <joint name="${tf_prefix}robotiq_85_left_knuckle_joint">
                 <command_interface name="position" />
-                <state_interface name="position" />
+                <state_interface name="position">
+                    <param name="initial_value">0.0</param>
+                </state_interface>
                 <state_interface name="velocity" />
             </joint>
+            <xacro:unless value="${use_fake_hardware}">
+                <gpio name="reactivate_gripper">
+                    <command_interface name="reactivate_gripper_cmd" />
+                    <command_interface name="reactivate_gripper_response" />
+                </gpio>
+            </xacro:unless>
         </ros2_control>
     </xacro:macro>

File: urdf/robotiq_gripper_macro.urdf.xacro (robot description, xacro)
@@ -1,11 +1,14 @@
 <?xml version="1.0"?>
 <robot xmlns:xacro="http://wiki.ros.org/xacro" name="robotiq_gripper">
-    <xacro:macro name="robotiq_gripper" params="parent *origin sim:=false tf_prefix">
-        <!-- ros2 control include -->
+    <xacro:macro name="robotiq_gripper" params="parent *origin sim:=false tf_prefix gripper_connection:=urcap com_port:=/dev/ttyUSB0 use_fake_hardware:=false">
         <xacro:include filename="$(find ur_description)/urdf/robotiq_gripper.ros2_control.xacro" />
-        <!-- ros2 control instance -->
-        <xacro:robotiq_gripper_ros2_control
-          name="robotiq_gripper_control"
-          com_port="/tmp/ttyUR"/>
+        <!-- URCap owns the tool serial port; only USB uses this hardware plugin. -->
+        <xacro:if value="${use_fake_hardware or gripper_connection == 'usb'}">
+          <xacro:robotiq_gripper_ros2_control
+            name="robotiq_gripper_control"
+            tf_prefix="${tf_prefix}"
+            com_port="${com_port}"
+            use_fake_hardware="${use_fake_hardware}"/>
+        </xacro:if>
         <link name="${tf_prefix}robotiq_85_base_link">
             <visual>

File: urdf/ur.urdf.xacro (robot description, xacro)
@@ -53,6 +53,8 @@
    <xacro:arg name="tool_device_name" default="/tmp/ttyUR" />
    <xacro:arg name="tool_tcp_port" default="54321" />
-   <!-- Flag to use the Gripper or just the UR5  -->
-   <xacro:arg name="use_gripper" default="true" />
+   <!-- Geometry is independent of the selected gripper connection. -->
+   <xacro:arg name="use_gripper" default="false" />
+   <xacro:arg name="gripper_connection" default="urcap" />
+   <xacro:arg name="gripper_port" default="/dev/ttyUSB0" />
    <!-- Flag to choose between custom gripper and robotiq gripper -->
    <xacro:arg name="use_custom_gripper" default="false" />
@@ -69,6 +71,4 @@
    <!-- Flag to preserve fixed joints and prevent lumping when generating SDF for Gazebo -->
    <xacro:arg name="gazebo_preserve_fixed_joint_arg" default="false"/>
-   <!-- Flag to use the Gripper or just the UR5  -->
-   <xacro:arg name="use_gripper" default="false" />
    <!-- initial position for simulations (Fake Hardware, Gazebo, Ignition) -->
    <xacro:arg name="initial_positions_file" default="$(find ur_description)/config/initial_positions.yaml"/>
@@ -106,4 +106,7 @@
         tf_prefix="$(arg tf_prefix)"
         parent="tool0"
+        gripper_connection="$(arg gripper_connection)"
+        com_port="$(arg gripper_port)"
+        use_fake_hardware="$(arg use_fake_hardware)"
       >
         <origin xyz="0.0 0.0 0.0" rpy="0 0 0"/>
